Commit message: change base link axis

File: resources/robots/meta_wl/urdf/meta_wl.urdf (robot description, URDF)
Before this commit: robot meta_wl, 7 links, 6 joints
Links:
- link base_link: mass 1.51004053175102 -> 1.65327950844393
- link l_foot: mass 0.394892486943145 -> 0.422534961029166
- link l_lower: mass 0.104306167055054 -> 0.178077513203325
- link l_upper: mass 0.032226200550069 -> 0.0344820345885739
- link r_foot: mass 0.394892486943146 -> 0.422534961029166
- link r_lower: mass 0.104306167055055 -> 0.265879317024864
- link r_upper: mass 0.032226200550069 -> 0.0344820345885739
Joints:
- joint l_hip: origin xyz=0 0 0 rpy=0 0 -2.3924 -> xyz=0.005 0 0 rpy=-1.5708 0.89586 1.5708
- joint l_knee: origin xyz=0.1566 0 0.00125 rpy=0 0 1.9355 -> xyz=0.1566 0 0.00125 rpy=0 0 1.6628
- joint l_wheel: origin xyz=0.1425 0 -0.0508 rpy=0 0 0.45687 -> xyz=0.1425 0 -0.0508 rpy=0 0 0.58297
- joint r_hip: origin xyz=0 0 0.242 rpy=0 0 -2.3924 -> xyz=-0.237 0 0 rpy=-1.5708 0.89586 1.5708
- joint r_knee: origin xyz=0.1566 0 -0.00125 rpy=0 0 1.9355 -> xyz=0.1566 0 -0.00125 rpy=0 0 1.6628
- joint r_wheel: origin xyz=0.1425 0 0.0508 rpy=0 0 0.45687 -> xyz=0.1425 0 0.0508 rpy=0 0 0.58297

Commit message: set zero pos in calc knee, solve bugs: meshes, enum, view

File: resources/robots/meta_wl/urdf/meta_wl.urdf (robot description, URDF)
Before this commit: robot meta_wl, 7 links, 6 joints
Links:
- link base_link: geometry collision mesh filename=../meshes/base_link.STL; visual mesh filename=../meshes/base_link.STL
- link l_foot: geometry collision mesh filename=../meshes/l_foot.STL; visual mesh filename=../meshes/l_foot.STL
- link l_lower: geometry collision mesh filename=../meshes/l_lower.STL; visual mesh filename=../meshes/l_lower.STL
- link l_upper: geometry collision mesh filename=../meshes/l_upper.STL; visual mesh filename=../meshes/l_upper.STL
- link r_foot: geometry collision mesh filename=../meshes/r_foot.STL; visual mesh filename=../meshes/r_foot.STL
- link r_lower: geometry collision mesh filename=../meshes/r_lower.STL; visual mesh filename=../meshes/r_lower.STL
- link r_upper: geometry collision mesh filename=../meshes/r_upper.STL; visual mesh filename=../meshes/r_upper.STL

Commit message: add joint limits to urdf

File: resources/robots/meta_wl/urdf/meta_wl.urdf (robot description, URDF)
Before this commit: robot meta_wl, 7 links, 6 joints
Joints:
- joint l_hip: limit lower=0 upper=0 effort=0 velocity=0 -> lower=-0.436 upper=0.262 effort=0 velocity=0
- joint l_knee: limit lower=0 upper=0 effort=0 velocity=0 -> lower=-0.53793 upper=0.83588 effort=0 velocity=0
- joint r_hip: limit lower=0 upper=0 effort=0 velocity=0 -> lower=-0.436 upper=0.262 effort=0 velocity=0
- joint r_knee: limit lower=0 upper=0 effort=0 velocity=0 -> lower=-0.53793 upper=0.83588 effort=0 velocity=0

Commit message: rename stl and successfully load the robot into gym, although it's bouncing

File: resources/robots/meta_wl/urdf/meta_wl.urdf (robot description, URDF)
Before this commit: robot meta_wl, 7 links, 6 joints
Links:
- removed link base_link
- removed link l_lower
- removed link l_upper
- removed link r_lower
- removed link r_upper
- added link base, mass 1.65327950844393; collision mesh filename=../meshes/base.STL; visual mesh filename=../meshes/base.STL
- added link l_shin, mass 0.178077513203325; collision mesh filename=../meshes/l_shin.STL; visual mesh filename=../meshes/l_shin.STL
- added link l_thigh, mass 0.0344820345885739; collision mesh filename=../meshes/l_thigh.STL; visual mesh filename=../meshes/l_thigh.STL
- added link r_shin, mass 0.265879317024864; collision mesh filename=../meshes/r_shin.STL; visual mesh filename=../meshes/r_shin.STL
- added link r_thigh, mass 0.0344820345885739; collision mesh filename=../meshes/r_thigh.STL; visual mesh filename=../meshes/r_thigh.STL
Joints:
- joint l_hip: child l_upper -> l_thigh; limit lower=-0.436 upper=0.262 effort=0 velocity=0 -> lower=-0.436 upper=0.262 effort=30 velocity=1000; parent base_link -> base
- joint l_knee: child l_lower -> l_shin; limit lower=-0.53793 upper=0.83588 effort=0 velocity=0 -> lower=-0.53793 upper=0.83588 effort=30 velocity=1000; parent l_upper -> l_thigh
- joint l_wheel: limit lower=0 upper=0 effort=0 velocity=0 -> effort=5 velocity=1000; parent l_lower -> l_shin
- joint r_hip: child r_upper -> r_thigh; limit lower=-0.436 upper=0.262 effort=0 velocity=0 -> lower=-0.436 upper=0.262 effort=30 velocity=1000; parent base_link -> base
- joint r_knee: child r_lower -> r_shin; limit lower=-0.53793 upper=0.83588 effort=0 velocity=0 -> lower=-0.53793 upper=0.83588 effort=30 velocity=1000; parent r_upper -> r_thigh
- joint r_wheel: limit lower=0 upper=0 effort=0 velocity=0 -> effort=5 velocity=1000; parent r_lower -> r_shin

Commit message: update urdf inertia and fix pd controller bug

File: resources/robots/meta_wl/urdf/meta_wl.urdf (robot description, URDF)
Before this commit: robot meta_wl, 7 links, 6 joints
Links:
- link base: mass 1.65327950844393 -> 3.385
- link r_shin: mass 0.265879317024864 -> 0.470

Commit message: update urdf inertia, look better now

File: resources/robots/meta_wl/urdf/meta_wl.urdf (robot description, URDF)
Before this commit: robot meta_wl, 7 links, 6 joints
Links:
- link base: mass 3.385 -> 3.422
- link l_foot: mass 0.422534961029166 -> 0.363247599426668
- link l_shin: mass 0.178077513203325 -> 0.086125018064217
- link r_foot: mass 0.422534961029166 -> 0.363247599426668
- link r_shin: mass 0.470 -> 0.0861250180642172
- link r_thigh: mass 0.0344820345885739 -> 0.0344820345885738
Joints:
- joint l_hip: origin xyz=0.005 0 0 rpy=-1.5708 0.89586 1.5708 -> xyz=-0.02 0.121 0.066 rpy=-1.5708 0.816 -3.1416
- joint l_knee: limit lower=-0.53793 upper=0.83588 effort=30 velocity=1000 -> lower=-0.538 upper=0.836 effort=30 velocity=1000; origin xyz=0.1566 0 0.00125 rpy=0 0 1.6628 -> xyz=0.1566 0 0.00125 rpy=0 0 1.8118
- joint l_wheel: origin xyz=0.1425 0 -0.0508 rpy=0 0 0.58297 -> xyz=0.1425 0 -0.0508 rpy=0 0 0.51383
- joint r_hip: origin xyz=-0.237 0 0 rpy=-1.5708 0.89586 1.5708 -> xyz=-0.02 -0.121 0.066 rpy=-1.5708 0.816 3.1416
- joint r_knee: limit lower=-0.53793 upper=0.83588 effort=30 velocity=1000 -> lower=-0.538 upper=0.836 effort=30 velocity=1000; origin xyz=0.1566 0 -0.00125 rpy=0 0 1.6628 -> xyz=0.1566 0 -0.00125 rpy=0 0 1.8118
- joint r_wheel: origin xyz=0.1425 0 0.0508 rpy=0 0 0.58297 -> xyz=0.1425 0 0.0508 rpy=0 0 0.51383

Commit message: change to use theta and leg

File: resources/robots/meta_wl/urdf/meta_wl.urdf (robot description, URDF)
Before this commit: robot meta_wl, 7 links, 6 joints
Links:
- link l_shin: mass 0.086125018064217 -> 0.528
- link r_shin: mass 0.0861250180642172 -> 0.528

Commit message: replace urdf with new prismatic ver, update vmc accordingly

File: resources/robots/meta_wl/urdf/meta_wl.urdf (robot description, URDF)
Before this commit: robot meta_wl, 7 links, 6 joints
Links:
- removed link base
- removed link l_foot
- removed link l_shin
- removed link l_thigh
- removed link r_foot
- removed link r_shin
- removed link r_thigh
- added link base_link, mass 3.422; collision mesh filename=../meshes/base_link.STL; visual mesh filename=../meshes/base_link.STL
- added link l_leg_link, mass 0.205618463841969; collision mesh filename=../meshes/l_leg_link.STL; visual mesh filename=../meshes/l_leg_link.STL
- added link l_wheel_link, mass 0.363247599426668; collision mesh filename=../meshes/l_wheel_link.STL; visual mesh filename=../meshes/l_wheel_link.STL
- added link r_leg_link, mass 0.205618464210299; collision mesh filename=../meshes/r_leg_link.STL; visual mesh filename=../meshes/r_leg_link.STL
- added link r_wheel_link, mass 0.363247599426668; collision mesh filename=../meshes/r_wheel_link.STL; visual mesh filename=../meshes/r_wheel_link.STL
Joints:
- removed joint l_hip
- removed joint l_knee
- removed joint l_wheel
- removed joint r_hip
- removed joint r_knee
- removed joint r_wheel
- added joint l_leg_joint: type prismatic, parent base_link, child l_leg_link, origin xyz=-0.02 0.121 0.066 rpy=-1.5708 1.0033 3.1416, axis 0.72714 0.68649 0, limit lower=-0.436 upper=0.262 effort=30 velocity=1000
- added joint l_wheel_joint: type continuous, parent l_leg_link, child l_wheel_link, origin xyz=0.17292 0.14156 -0.04955 rpy=0 0 2.1383, axis 0 0 1
- added joint r_leg_joint: type prismatic, parent base_link, child r_leg_link, origin xyz=-0.02 -0.116 0.066 rpy=-1.5708 1.0033 3.1416, axis 0.72714 0.68649 0, limit lower=-0.436 upper=0.262 effort=30 velocity=1000
- added joint r_wheel_joint: type continuous, parent r_leg_link, child r_wheel_link, origin xyz=0.17292 0.14156 0.05455 rpy=0 0 2.1383, axis 0 0 1

Commit message: update urdf limits

File: resources/robots/meta_wl/urdf/meta_wl.urdf (robot description, URDF)
Before this commit: robot meta_wl, 5 links, 4 joints
Joints:
- joint l_leg_joint: limit lower=-0.436 upper=0.262 effort=30 velocity=1000 -> lower=-0.125 upper=0.035 effort=100 velocity=1000
- joint l_wheel_joint: limit (none) -> effort=5 velocity=1000
- joint r_leg_joint: limit lower=-0.436 upper=0.262 effort=30 velocity=1000 -> lower=-0.125 upper=0.035 effort=100 velocity=1000
- joint r_wheel_joint: limit (none) -> effort=5 velocity=1000

Commit message: add a frame to the robot, training looks better

File: resources/robots/meta_wl/urdf/meta_wl.urdf (robot description, URDF)
Before this commit: robot meta_wl, 5 links, 4 joints
Links:
- link l_leg_link: mass 0.205618463841969 -> 0.20607138537343
- link r_leg_link: mass 0.205618464210299 -> 0.206071385741738
Joints:
- joint l_leg_joint: axis 0.72714 0.68649 0 -> 0.56085 0.82792 0; origin xyz=-0.02 0.121 0.066 rpy=-1.5708 1.0033 3.1416 -> xyz=-0.00053949 0.12101 0.071375 rpy=-1.5708 0.59541 -3.1416
- joint l_wheel_joint: origin xyz=0.17292 0.14156 -0.04955 rpy=0 0 2.1383 -> xyz=0.1146 0.13617 -0.04955 rpy=0 0 2.357; type continuous -> revolute
- joint r_leg_joint: axis 0.72714 0.68649 0 -> 0.56085 0.82792 0; origin xyz=-0.02 -0.116 0.066 rpy=-1.5708 1.0033 3.1416 -> xyz=-0.00053949 -0.11599 0.071375 rpy=-1.5708 0.59541 3.1416
- joint r_wheel_joint: origin xyz=0.17292 0.14156 0.05455 rpy=0 0 2.1383 -> xyz=0.1146 0.13617 0.05455 rpy=0 0 2.357; type continuous -> revolute

Commit message: rotate ang vel and tune params

File: resources/robots/meta_wl/urdf/meta_wl.urdf (robot description, URDF)
Before this commit: robot meta_wl, 5 links, 4 joints
Links:
- link base_link: mass 3.422 -> 3.78
Joints:
- joint l_wheel_joint: limit effort=5 velocity=1000 -> effort=50 velocity=1000
- joint r_wheel_joint: limit effort=5 velocity=1000 -> effort=50 velocity=1000

Commit message: add base with no frame

File: resources/robots/meta_wl/urdf/meta_wl.urdf (robot description, URDF)
Before this commit: robot meta_wl, 5 links, 4 joints
Links:
- link l_leg_link: mass 0.20607138537343 -> 0.384
- link r_leg_link: mass 0.206071385741738 -> 0.384

Commit message: update inertia and add penalty on leg acc

File: resources/robots/meta_wl/urdf/meta_wl.urdf (robot description, URDF)
Before this commit: robot meta_wl, 5 links, 4 joints
Links:
- link l_leg_link: mass 0.384 -> 0.4
- link l_wheel_link: mass 0.363247599426668 -> 0.1
- link r_leg_link: mass 0.384 -> 0.4
- link r_wheel_link: mass 0.363247599426668 -> 0.1
